Commit message: Changed ur-URDF file

File: ws_moveit2/src/robo_planner/config/share/ur_description/urdf/ur_macro.xacro (robot description, xacro)
@@ -258,12 +258,14 @@
       <visual>
         <geometry>
-	    <box size="0.1 0.1 0.3"/>
-        </geometry>
-        <origin xyz="0 0 0.1501" rpy="0 0 0"/>
-      </visual>
-      <collision>
-        <origin xyz="0 0 0.1501" rpy="0 0 0"/>
-        <geometry>
-	    <box size="0.1 0.1 0.3"/>
+            <!--<box size="0.0 0.0 0.0"/>-->
+	    <box size="0.1 0.1 0.2"/>
+        </geometry>
+        <origin xyz="0 0 0.1" rpy="0 0 0"/>
+      </visual>
+      <collision>
+        <origin xyz="0 0 0.1" rpy="0 0 0"/>
+        <geometry>
+            <box size="0 0 0"/>
+	    <!--<box size="0.1 0.1 0.2"/>-->
         </geometry>
       </collision>
@@ -273,10 +275,14 @@
         <geometry>
 	        <box size="0.075 0.14 0.03"/>
-        </geometry>
+	        <!--<box size="0.0 0.0 0.0"/>-->
+        </geometry>
+          <!--<origin xyz="-0.03 0.13 -0.1" rpy="0 0 0"/>-->
           <origin xyz="-0.031 0.118 -0.018" rpy="0 0 0"/>
       </visual>
       <collision>
+        <!--<origin xyz="-0.03 0.13 -0.1" rpy="0 0 0"/>-->
         <origin xyz="-0.031 0.118 -0.018" rpy="0 0 0"/>
         <geometry>
+	        <!--<box size="0.0 0.0 0.0"/>-->
 	        <box size="0.075 0.14 0.03"/>
         </geometry>

Commit message: Added cable conduit do URDF file

File: ws_moveit2/src/robo_planner/config/share/ur_description/urdf/ur_macro.xacro (robot description, xacro)
@@ -274,16 +274,34 @@
       <visual>
         <geometry>
-	        <box size="0.075 0.14 0.03"/>
+	        <box size="0.014 0.14 0.008"/>
 	        <!--<box size="0.0 0.0 0.0"/>-->
         </geometry>
           <!--<origin xyz="-0.03 0.13 -0.1" rpy="0 0 0"/>-->
-          <origin xyz="-0.031 0.118 -0.018" rpy="0 0 0"/>
+          <origin xyz="0 0.118 -0.012" rpy="0 0 0"/>
       </visual>
       <collision>
         <!--<origin xyz="-0.03 0.13 -0.1" rpy="0 0 0"/>-->
-        <origin xyz="-0.031 0.118 -0.018" rpy="0 0 0"/>
+        <origin xyz="0 0.118 -0.012" rpy="0 0 0"/>
         <geometry>
 	        <!--<box size="0.0 0.0 0.0"/>-->
-	        <box size="0.075 0.14 0.03"/>
+	        <box size="0.014 0.14 0.008"/>
+        </geometry>
+      </collision>
+    </link>
+    <link name="${tf_prefix}cable_conduit_link">
+      <visual>
+        <geometry>
+	        <box size="0.06 0.06 0.06"/>
+	        <!--<box size="0.0 0.0 0.0"/>-->
+        </geometry>
+          <!--<origin xyz="-0.03 0.13 -0.1" rpy="0 0 0"/>-->
+          <origin xyz="-0.038 0.156 -0.028" rpy="0 0 0"/>
+      </visual>
+      <collision>
+        <!--<origin xyz="-0.03 0.13 -0.1" rpy="0 0 0"/>-->
+        <origin xyz="-0.038 0.156 -0.028" rpy="0 0 0"/>
+        <geometry>
+	        <!--<box size="0.0 0.0 0.0"/>-->
+	        <box size="0.06 0.06 0.06"/>
         </geometry>
       </collision>
@@ -386,4 +404,9 @@
       <parent link="${tf_prefix}tool0"/>
       <child link="${tf_prefix}cable_mount_link"/>
+      <origin xyz="0 0 0" rpy="0 0 0"/>
+    </joint>
+    <joint name="${tf_prefix}cable_conduit_joint" type="fixed">
+      <parent link="${tf_prefix}tool0"/>
+      <child link="${tf_prefix}cable_conduit_link"/>
       <origin xyz="0 0 0" rpy="0 0 0"/>
     </joint>

Commit message: Clean ur_pliz package Create neu launchfile Update readme Update urdf Fix parameters not correctly being loaded Cleanup and refactoring of scheduler

File: ws_moveit2/src/robo_planner/config/share/ur_description/urdf/ur_macro.xacro (robot description, xacro)
@@ -259,12 +259,14 @@
         <geometry>
             <!--<box size="0.0 0.0 0.0"/>-->
-	    <box size="0.1 0.1 0.2"/>
-        </geometry>
-        <origin xyz="0 0 0.1" rpy="0 0 0"/>
-      </visual>
-      <collision>
-        <origin xyz="0 0 0.1" rpy="0 0 0"/>
-        <geometry>
-            <box size="0 0 0"/>
+	    <!--<box size="0.1 0.1 0.3"/>-->
+	    <cylinder length="0.3" radius="0.05"/>
+        </geometry>
+        <origin xyz="0 0 0.1501" rpy="0 0 0"/>
+      </visual>
+      <collision>
+        <origin xyz="0 0 0.1501" rpy="0 0 0"/>
+        <geometry>
+            <!--<box size="0.1 0.1 0.3"/>-->
+            <cylinder length="0.3" radius="0.05"/>
 	    <!--<box size="0.1 0.1 0.2"/>-->
         </geometry>

Commit message: Collision Box of Endeffector smaller - All carrier positions are now implemented - BEMI 2 ist implemented - implemented taskPickPC1 funktion

File: ws_moveit2/src/robo_planner/config/share/ur_description/urdf/ur_macro.xacro (robot description, xacro)
@@ -255,30 +255,57 @@
       </xacro:cylinder_inertial>
     </link>
-    <link name="${tf_prefix}gripper_link">
+    <link name="${tf_prefix}gripper_link_upper">
       <visual>
         <geometry>
             <!--<box size="0.0 0.0 0.0"/>-->
 	    <!--<box size="0.1 0.1 0.3"/>-->
-	    <cylinder length="0.3" radius="0.05"/>
-        </geometry>
-        <origin xyz="0 0 0.1501" rpy="0 0 0"/>
-      </visual>
-      <collision>
-        <origin xyz="0 0 0.1501" rpy="0 0 0"/>
+	    <cylinder length="0.22" radius="0.045"/>
+        </geometry>
+        <origin xyz="0 0 0.1102" rpy="0 0 0"/>
+        <material name="grau">
+            <color rgba="0.365 0.37 0.388 1.0"/>
+        </material>
+      </visual>
+      <collision>
+        <origin xyz="0 0 0.1102" rpy="0 0 0"/>
         <geometry>
             <!--<box size="0.1 0.1 0.3"/>-->
-            <cylinder length="0.3" radius="0.05"/>
+            <cylinder length="0.22" radius="0.045"/>
 	    <!--<box size="0.1 0.1 0.2"/>-->
         </geometry>
       </collision>
     </link>
+    <link name="${tf_prefix}gripper_link_lower">
+      <visual>
+        <geometry>
+            <!--<box size="0.0 0.0 0.0"/>-->
+	    <!--<box size="0.1 0.1 0.3"/>-->
+	    <cylinder length="0.10" radius="0.014"/>
+        </geometry>
+        <origin xyz="0 0 0.2704" rpy="0 0 0"/>
+	<material name="grau">
+            <color rgba="0.365 0.37 0.388 1.0"/>
+        </material>
+      </visual>
+      <collision>
+        <origin xyz="0 0 0.2704" rpy="0 0 0"/>
+        <geometry>
+            <!--<box size="0.1 0.1 0.3"/>-->
+            <cylinder length="0.10" radius="0.014"/>
+	    <!--<box size="0.1 0.1 0.2"/>-->
+        </geometry>
+      </collision>
+    </link>
     <link name="${tf_prefix}cable_mount_link">
       <visual>
         <geometry>
-	        <box size="0.014 0.14 0.008"/>
+	        <box size="0.02 0.14 0.015"/>
 	        <!--<box size="0.0 0.0 0.0"/>-->
         </geometry>
           <!--<origin xyz="-0.03 0.13 -0.1" rpy="0 0 0"/>-->
           <origin xyz="0 0.118 -0.012" rpy="0 0 0"/>
+	<material name="grau">
+            <color rgba="0.365 0.37 0.388 1.0"/>
+        </material>
       </visual>
       <collision>
@@ -287,5 +314,5 @@
         <geometry>
 	        <!--<box size="0.0 0.0 0.0"/>-->
-	        <box size="0.014 0.14 0.008"/>
+	        <box size="0.02 0.14 0.015"/>
         </geometry>
       </collision>
@@ -294,9 +321,12 @@
       <visual>
         <geometry>
-	        <box size="0.06 0.06 0.06"/>
+	        <box size="0.055 0.06 0.06"/>
 	        <!--<box size="0.0 0.0 0.0"/>-->
         </geometry>
           <!--<origin xyz="-0.03 0.13 -0.1" rpy="0 0 0"/>-->
           <origin xyz="-0.038 0.156 -0.028" rpy="0 0 0"/>
+	<material name="grau">
+            <color rgba="0.365 0.37 0.388 1.0"/>
+        </material>
       </visual>
       <collision>
@@ -305,5 +335,5 @@
         <geometry>
 	        <!--<box size="0.0 0.0 0.0"/>-->
-	        <box size="0.06 0.06 0.06"/>
+	        <box size="0.055 0.06 0.06"/>
         </geometry>
       </collision>
@@ -398,7 +428,12 @@
       <dynamics damping="0" friction="0"/>
     </joint>
-    <joint name="${tf_prefix}gripper_joint" type="fixed">
+    <joint name="${tf_prefix}gripper_joint_upper" type="fixed">
       <parent link="${tf_prefix}tool0"/>
-      <child link="${tf_prefix}gripper_link"/>
+      <child link="${tf_prefix}gripper_link_upper"/>
+      <origin xyz="0 0 0" rpy="0 0 0"/>
+    </joint>
+    <joint name="${tf_prefix}gripper_joint_lower" type="fixed">
+      <parent link="${tf_prefix}tool0"/>
+      <child link="${tf_prefix}gripper_link_lower"/>
       <origin xyz="0 0 0" rpy="0 0 0"/>
     </joint>
